File: sra_dev_board_2022/sra_dev_board_2022.kicad_sch (KiCad schematic)
At the start: 78 parts, among them J1 Conn_01x19_Male, J10 Conn_01x03_Male, J11 Conn_01x05_Male, J12 Conn_01x05_Male, J13 Conn_01x05_Male, J2 Conn_01x03_Male, J3 Conn_01x03_Male, J4 Conn_01x03_Male, J5 Conn_01x19_Male, J6 DCJ200-10-A-XX-X_REVA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

Commit message: Added drv8825 stepper motor driver
Parts:
- removed R15, R16, R17, R18: 1k, Resistor_SMD:R_1206_3216Metric, symbol Device:R
- removed T2: Screw_Terminal_01x04, terminal_block:motor_1x04_tht, symbol Connector:Screw_Terminal_01x04
- removed U4: TB6612FNG, motor_driver:TB6612FNG_2, symbol TB6612FNG:ROB-14450
- added A1: drv8825, motor_driver:IC_DRV8825_STEPPER_MOTOR_DRIVER_CARRIER, symbol drv8825:drv8825
- added C7: 100uF, Capacitor_SMD:CP_Elec_6.3x7.7, symbol Device:C_Polarized_Small
- added J14, J16: Conn_01x03_Male, Connector_PinHeader_2.54mm:PinHeader_1x03_P2.54mm_Vertical, symbol Connector:Conn_01x03_Male
- added J15: Conn_01x04_Male, Connector_PinHeader_2.54mm:PinHeader_1x04_P2.54mm_Vertical, symbol Connector:Conn_01x04_Male
Connections:
- net 12: now also A1.7 (STEP)
- net 12V_U: now also A1.16 (VMOT), C7.1
- net 13: now also A1.8 (DIR)
- net 14: no longer TB_B1.5 (B)
- net 27: no longer TB_B1.2 (B)
- net 3V3: no longer U3.10 (PWMB), U3.13 (STBY), U3.16 (PWMA)
- net 5V_P: now also A1.5 (~{RST}), A1.6 (~{SLP}), J14.1 (Pin_1), J14.2 (Pin_2), J14.3 (Pin_3)
- net GND: now also A1.1 (~{EN}), A1.15 (GND_MOT), A1.9 (GND_LOGIC), C7.2
- net OUT1B: now also A1.14 (B2), J15.1 (Pin_1)
- net OUT2B: now also A1.13 (B1), J15.2 (Pin_2)
- net OUT3B: now also A1.12 (A1), J15.3 (Pin_3)
- net OUT4B: now also A1.11 (A2), J15.4 (Pin_4)
- net at R11.2: no longer U3.14 (AI1)
- net at U3.11 (BI2): no longer R14.2
- net at U3.12 (BI1): no longer R13.2
- net at U3.15 (AI2): no longer R12.2
- new net BIN1: TB_B1.2 (B)
- new net BIN2: TB_B1.5 (B)
- new net M0: A1.2 (M0), J16.1 (Pin_1)
- new net M1: A1.3 (M1), J16.2 (Pin_2)
- new net M2: A1.4 (M2), J16.3 (Pin_3)
Other:
- moved on the sheet: R11, R12, R13, R14, U3
